File: hardware/io.kicad_sch (KiCad schematic)
At the start: 3 parts, among them U8 PCA9534PWR

Commit message: t
Parts:
- removed C78: 100n, Capacitor_SMD:C_0603_1608Metric, symbol Device:C
- removed R53: 10k, Resistor_SMD:R_0603_1608Metric, symbol Device:R
- removed U8: PCA9534PWR, general:SOP65P640X120-16N, symbol general:PCA9534PWR
- added C25: 100n, Capacitor_SMD:C_0603_1608Metric, symbol Device:C
- added D3, D4: LED_GREEN, general:LED_3210Metric_Right_Angle, symbol Device:LED
- added D5, D6: LED_BLUE, general:LED_3210Metric_Right_Angle, symbol Device:LED
- added J2: SHF-108-01-L-D-SM, SHF-108-01-X-D-SM, symbol general:SHF-108-01-L-D-SM
- added J3: SHF-103-01-L-D-SM, general:SAMTEC_SHF-103-01-L-D-SM, symbol general:SHF-103-01-L-D-SM
- added R22, R23: 1.5k, Resistor_SMD:R_0603_1608Metric, symbol Device:R
- added TP1: 12V, TestPoint:TestPoint_Pad_D2.0mm, symbol Connector:TestPoint_Small
- added TP2: 3.3V, TestPoint:TestPoint_Pad_D2.0mm, symbol Connector:TestPoint_Small
- added TP3: GND, TestPoint:TestPoint_Pad_D2.0mm, symbol Connector:TestPoint_Small
- added U3: PCA9536TK, general:SON50P300X300X100-9N-D, symbol Interface_Expansion:PCA9536D
Connections:
- net +3.3V: now also C25.1, J2.2, J3.2, TP2.1, U3.8 (VDD)
- net GND: now also C25.2, D3.1 (K), D4.1 (K), D5.1 (K), D6.1 (K), J2.3, J3.4, TP3.1, U3.4 (VSS)
- new net: D3.2 (A), D4.2 (A), R22.2
- new net: D5.2 (A), D6.2 (A), R23.2
- new net +12V: J2.1, TP1.1
- new net ESP_EN: J3.1
- new net GPI34: J2.13
- new net GPI35: J2.14
- new net GPIO0: J3.6
- new net GPIO12_I2C_SCL: J2.7, U3.6 (SCL)
- new net GPIO13_I2C_SDA: J2.8, U3.7 (SDA)
- new net GPIO14: J2.9
- new net GPIO15: J2.10
- new net GPIO2: J2.4
- new net GPIO32: J2.11
- new net GPIO33: J2.12
- new net GPIO4: J2.5
- new net GPIO5: J2.6
- new net I2C_GPIO1: J2.15, U3.3 (IO2)
- new net I2C_GPIO2: J2.16, U3.5 (IO3)
- new net LED1: R22.1, U3.1 (IO0)
- new net LED2: R23.1, U3.2 (IO1)
- new net RXD0: J3.5
- new net TXD0: J3.3
- no-connect marks 4 -> 0
